Commit message: add base_footprint and a fixed joint

File: urdf/simple_car.urdf (robot description, URDF)
Before this commit: robot simple_car, 5 links, 4 joints
Links:
- added link base_footprint
Joints:
- added joint fixed: type fixed, parent base_footprint, child base_link, origin xyz=0 0 0.005 rpy=0 0 0
